File: hardware/eurorack-pmod-r3.3/led_driver.kicad_sch (KiCad schematic)
At the start: 23 parts, among them U10 PCA9635 LED DRIVER

Commit message: - Swap all tantalums for ceramics
Parts:
- C28: value 100.0uF -> 22.0uF; footprint Capacitor_Tantalum_SMD:CP_EIA-3216-10_Kemet-I -> Capacitor_SMD:C_1206_3216Metric; lcsc# C27279 -> C12891
Changed lines of the file:
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@@
 			)
 		)
-		(property "Value" "100.0uF"
+		(property "Value" "22.0uF"
 			(at 58.42 77.47 0)
 			(effects
@@
 			)
 		)
-		(property "Footprint" "Capacitor_Tantalum_SMD:CP_EIA-3216-10_Kemet-I"
+		(property "Footprint" "Capacitor_SMD:C_1206_3216Metric"
 			(at 63.5 77.47 0)
 			(effects
@@
 			)
 		)
-		(property "lcsc#" "C27279"
+		(property "lcsc#" "C12891"
 			(at 63.5 77.47 0)
 			(effects
