File: hardware/eurorack-pmod-r3.3/dual_mono_inputs.kicad_sch (KiCad schematic)
At the start: 13 parts, among them J4 AUDIO JACK PJ-324M0, J5 AUDIO JACK PJ-324M0, U3 TL074 OP AMP

Commit message: - Add ceradiodes to audio ins/outs - Add low-capacitance TVS to touch channels (TODO footprint)
Parts:
- added D27, D29: LLP1006-2M, symbol Device:D_TVS_Small_Filled
- added RV1, RV3: Ceradiode 65V, Capacitor_SMD:C_0603_1608Metric, symbol Device:Varistor
Connections:
- net CAP_SENSE1: now also D27.2 (A2)
- net CAP_SENSE2: now also D29.2 (A2)
- net GND: now also D27.1 (A1), D29.1 (A1), RV1.2, RV3.2
- net at J4.T, R6.1: now also RV1.1
- net at J5.T, R9.1: now also RV3.1

Commit message: - ceradiodes/tvs: place and route
Parts:
- D27, D29: value LLP1006-2M -> VBUS05L1; footprint (none) -> LLP1006-2M:VISHAY-LLP1006-2M
Changed lines of the file:
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@@
 			)
 		)
-		(property "Value" "LLP1006-2M"
+		(property "Value" "VBUS05L1"
 			(at 35.56 50.7999 90)
 			(effects
@@
 			)
 		)
-		(property "Footprint" ""
+		(property "Footprint" "LLP1006-2M:VISHAY-LLP1006-2M"
 			(at 33.02 49.53 0)
 			(effects
@@
 			)
 		)
-		(property "Value" "LLP1006-2M"
+		(property "Value" "VBUS05L1"
 			(at 34.29 118.1099 90)
 			(effects
@@
 			)
 		)
-		(property "Footprint" ""
+		(property "Footprint" "LLP1006-2M:VISHAY-LLP1006-2M"
 			(at 31.75 116.84 0)
 			(effects

Commit message: vref: replace +3.0V with local 12V->3.3V LDO
Connections:
- net +3.3VA renamed VDD
Changed lines of the file:
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@@
-	)
-	(symbol
-		(lib_id "power:+3.3VA")
-		(at 41.91 88.9 0)
-		(mirror y)
-		(unit 1)
-		(exclude_from_sim no)
-		(in_bom yes)
-		(on_board yes)
-		(dnp no)
-		(property "Reference" "#PWR067"
-			(at 41.91 92.71 0)
-			(effects
-				(font
-					(size 1.27 1.27)
-				)
-				(hide yes)
-			)
-		)
-		(property "Value" "+3.3VA"
-			(at 40.64 85.09 0)
-			(effects
-				(font
-					(size 1.27 1.27)
-				)
-			)
-		)
-		(property "Footprint" ""
-			(at 41.91 88.9 0)
-			(effects
-				(font
-					(size 1.27 1.27)
-				)
-				(hide yes)
-			)
-		)
-		(property "Datasheet" ""
-			(at 41.91 88.9 0)
-			(effects
-				(font
-					(size 1.27 1.27)
-				)
-				(hide yes)
-			)
-		)
-		(property "Description" ""
-			(at 41.91 88.9 0)
-			(effects
-				(font
-					(size 1.27 1.27)
-				)
-			)
-		)
-		(pin "1"
-		)
-		(instances
-			(project "eurorack-pmod-pcb"
-				(path "/d1469efb-590b-4a61-a37b-5bbc286936ba/26ad21f7-706e-4aa7-ae23-d7556e7daddf"
-					(reference "#PWR075")
-					(unit 1)
-				)
-				(path "/d1469efb-590b-4a61-a37b-5bbc286936ba/ffd79913-d69b-48e3-a2e5-4374ac43aecb"
-					(reference "#PWR067")
-					(unit 1)
-				)
-			)
-		)
 	)
 	(symbol
@@
 				(path "/d1469efb-590b-4a61-a37b-5bbc286936ba/ffd79913-d69b-48e3-a2e5-4374ac43aecb"
 					(reference "#PWR0123")
-					(unit 1)
-				)
-			)
-		)
-	)
-	(symbol
-		(lib_id "power:+3.3VA")
-		(at 43.18 20.32 0)
-		(mirror y)
-		(unit 1)
-		(exclude_from_sim no)
-		(in_bom yes)
-		(on_board yes)
-		(dnp no)
-		(property "Reference" "#PWR063"
-			(at 43.18 24.13 0)
-			(effects
-				(font
-					(size 1.27 1.27)
-				)
-				(hide yes)
-			)
-		)
-		(property "Value" "+3.3VA"
-			(at 41.91 16.51 0)
-			(effects
-				(font
-					(size 1.27 1.27)
-				)
-			)
-		)
-		(property "Footprint" ""
-			(at 43.18 20.32 0)
-			(effects
-				(font
-					(size 1.27 1.27)
-				)
-				(hide yes)
-			)
-		)
-		(property "Datasheet" ""
-			(at 43.18 20.32 0)
-			(effects
-				(font
-					(size 1.27 1.27)
-				)
-				(hide yes)
-			)
-		)
-		(property "Description" ""
-			(at 43.18 20.32 0)
-			(effects
-				(font
-					(size 1.27 1.27)
-				)
-			)
-		)
-		(pin "1"
-		)
-		(instances
-			(project "eurorack-pmod-pcb"
-				(path "/d1469efb-590b-4a61-a37b-5bbc286936ba/26ad21f7-706e-4aa7-ae23-d7556e7daddf"
-					(reference "#PWR071")
-					(unit 1)
-				)
-				(path "/d1469efb-590b-4a61-a37b-5bbc286936ba/ffd79913-d69b-48e3-a2e5-4374ac43aecb"
-					(reference "#PWR063")
 					(unit 1)
 				)
@@
 	)
 	(symbol
+		(lib_id "power:VDD")
+		(at 41.91 88.9 0)
+		(unit 1)
+		(exclude_from_sim no)
+		(in_bom yes)
+		(on_board yes)
+		(dnp no)
+		(property "Reference" "#PWR067"
+			(at 41.91 92.71 0)
+			(effects
+				(font
+					(size 1.27 1.27)
+				)
+				(hide yes)
+			)
+		)
+		(property "Value" "VDD"
+			(at 41.91 84.963 0)
+			(effects
+				(font
+					(size 1.27 1.27)
+				)
+			)
+		)
+		(property "Footprint" ""
+			(at 41.91 88.9 0)
+			(effects
+				(font
+					(size 1.27 1.27)
+				)
+				(hide yes)
+			)
+		)
+		(property "Datasheet" ""
+			(at 41.91 88.9 0)
+			(effects
+				(font
+					(size 1.27 1.27)
+				)
+				(hide yes)
+			)
+		)
+		(property "Description" ""
+			(at 41.91 88.9 0)
+			(effects
+				(font
+					(size 1.27 1.27)
+				)
+			)
+		)
+		(pin "1"
+		)
+		(instances
+			(project "eurorack-pmod-pcb"
+				(path "/d1469efb-590b-4a61-a37b-5bbc286936ba/26ad21f7-706e-4aa7-ae23-d7556e7daddf"
+					(reference "#PWR075")
+					(unit 1)
+				)
+				(path "/d1469efb-590b-4a61-a37b-5bbc286936ba/ffd79913-d69b-48e3-a2e5-4374ac43aecb"
+					(reference "#PWR067")
+					(unit 1)
+				)
+			)
+		)
+	)
+	(symbol
 		(lib_id "Device:R")
 		(at 120.65 107.95 90)
@@
 					(unit 1)
 				)
+			)
+		)
+	)
+	(symbol
+		(lib_id "power:VDD")
+		(at 43.18 20.32 0)
+		(unit 1)
+		(exclude_from_sim no)
+		(in_bom yes)
+		(on_board yes)
+		(dnp no)
+		(property "Reference" "#PWR063"
+			(at 43.18 24.13 0)
+			(effects
+				(font
+					(size 1.27 1.27)
+				)
+				(hide yes)
+			)
+		)
+		(property "Value" "VDD"
+			(at 43.18 16.383 0)
+			(effects
+				(font
+					(size 1.27 1.27)
+				)
+			)
+		)
+		(property "Footprint" ""
+			(at 43.18 20.32 0)
+			(effects
+				(font
+					(size 1.27 1.27)
+				)
+				(hide yes)
+			)
+		)
+		(property "Datasheet" ""
+			(at 43.18 20.32 0)
+			(effects
+				(font
+					(size 1.27 1.27)
+				)
+				(hide yes)
+			)
+		)
+		(property "Description" ""
+			(at 43.18 20.32 0)
+			(effects
+				(font
+					(size 1.27 1.27)
+				)
+			)
+		)
+		(pin "1"
+		)
+		(instances
+			(project "eurorack-pmod-pcb"
+				(path "/d1469efb-590b-4a61-a37b-5bbc286936ba/26ad21f7-706e-4aa7-ae23-d7556e7daddf"
+					(reference "#PWR071")
+					(unit 1)
+				)
+				(path "/d1469efb-590b-4a61-a37b-5bbc286936ba/ffd79913-d69b-48e3-a2e5-4374ac43aecb"
+					(reference "#PWR063")
+					(unit 1)
+				)
